Commit message: Organizing files

File: webots_prometheus/protos/robot.urdf (robot description, URDF)
Before this commit: robot onshape, 21 links, 20 joints
Links:
- link braco: geometry collision mesh filename=/home/llagoeiro/Desktop/IC/IC-Prometheus-Webots/webots_prom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; collision mesh filename=/home/llagoeiro/Desktop/IC/IC-Prometheus-Webots/webots_prom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
- link braco_2: geometry collision mesh filename=/home/llagoeiro/Desktop/IC/IC-Prometheus-Webots/webots_prom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; collision mesh filename=/home/llagoeiro/Desktop/IC/IC-Prometheus-Webots/webots_prom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
- link canela: mass 0.19257782476461676735 -> 0.19257782476461682286; geometry collision mesh filename=/home/llagoeiro/Desktop/IC/IC-Prometheus-Webots/webots_prom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; visual mesh filename=/home/llagoeiro/Desktop/IC/IC-Prometheus-Webots/webots_prom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
- link canela_2: mass 0.19257782476461676735 -> 0.19257782476461682286; geometry collision mesh filename=/home/llagoeiro/Desktop/IC/IC-Prometheus-Webots/webots_prom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; visual mesh filename=/home/llagoeiro/Desktop/IC/IC-Prometheus-Webots/webots_prom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
- link capacete: geometry collision mesh filename=/home/llagoeiro/Desktop/IC/IC-Prometheus-Webots/webots_prom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; collision mesh filename=/home/llagoeiro/Desktop/IC/IC-Prometheus-Webots/webots_prom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
- link conector_calcanhar: mass 0.15254261535712484998 -> 0.15254261535712493325; geometry collision mesh filename=/home/llagoeiro/Desktop/IC/IC-Prometheus-Webots/webots_prom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; visual mesh filename=/home/llagoeiro/Desktop/IC/IC-Prometheus-Webots/webots_prom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
- link conector_calcanhar_2: mass 0.15254261535712484998 -> 0.15254261535712493325; geometry collision mesh filename=/home/llagoeiro/Desktop/IC/IC-Prometheus-Webots/webots_prom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; visual mesh filename=/home/llagoeiro/Desktop/IC/IC-Prometheus-Webots/webots_prom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
- link joelho: mass 0.8669178102972361355 -> 0.86691781029723602447; geometry collision mesh filename=/home/llagoeiro/Desktop/IC/IC-Prometheus-Webots/webots_prom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; collision mesh filename=/home/llagoeiro/Desktop/IC/IC-Prometheus-Webots/webots_prom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
- link joelho_2: mass 0.8669178102972361355 -> 0.86691781029723602447; geometry collision mesh filename=/home/llagoeiro/Desktop/IC/IC-Prometheus-Webots/webots_prom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; collision mesh filename=/home/llagoeiro/Desktop/IC/IC-Prometheus-Webots/webots_prom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
- link mao: geometry collision mesh filename=/home/llagoeiro/Desktop/IC/IC-Prometheus-Webots/webots_prom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; collision mesh filename=/home/llagoeiro/Desktop/IC/IC-Prometheus-Webots/webots_prom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
- link mao_2: geometry collision mesh filename=/home/llagoeiro/Desktop/IC/IC-Prometheus-Webots/webots_prom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; collision mesh filename=/home/llagoeiro/Desktop/IC/IC-Prometheus-Webots/webots_prom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
- link motores_duplos: geometry collision mesh filename=/home/llagoeiro/Desktop/IC/IC-Prometheus-Webots/webots_prom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; collision mesh filename=/home/llagoeiro/Desktop/IC/IC-Prometheus-Webots/webots_prom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
- link motores_duplos_2: mass 1.5325984925954143634 -> 1.5325984925954141413; geometry collision mesh filename=/home/llagoeiro/Desktop/IC/IC-Prometheus-Webots/webots_prom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; collision mesh filename=/home/llagoeiro/Desktop/IC/IC-Prometheus-Webots/webots_prom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
- link motores_duplos_3: geometry collision mesh filename=/home/llagoeiro/Desktop/IC/IC-Prometheus-Webots/webots_prom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; collision mesh filename=/home/llagoeiro/Desktop/IC/IC-Prometheus-Webots/webots_prom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
- link motores_duplos_4: mass 1.5325984925954145854 -> 1.5325984925954143634; geometry collision mesh filename=/home/llagoeiro/Desktop/IC/IC-Prometheus-Webots/webots_prom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; collision mesh filename=/home/llagoeiro/Desktop/IC/IC-Prometheus-Webots/webots_prom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
- link ombro: mass 0.059819249656771315837 -> 0.059819249656771308898; geometry collision mesh filename=/home/llagoeiro/Desktop/IC/IC-Prometheus-Webots/webots_prom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; visual mesh filename=/home/llagoeiro/Desktop/IC/IC-Prometheus-Webots/webots_prom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
- link ombro_2: mass 0.059819249656771315837 -> 0.059819249656771308898; geometry collision mesh filename=/home/llagoeiro/Desktop/IC/IC-Prometheus-Webots/webots_prom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; visual mesh filename=/home/llagoeiro/Desktop/IC/IC-Prometheus-Webots/webots_prom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
- link pe_direito: mass 0.23919353074394250624 -> 0.23919353074394258951; geometry collision mesh filename=/home/llagoeiro/Desktop/IC/IC-Prometheus-Webots/webots_prom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; collision mesh filename=/home/llagoeiro/Desktop/IC/IC-Prometheus-Webots/webots_prom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
- link pe_esquerdo: mass 0.23919353074394250624 -> 0.23919353074394258951; geometry collision mesh filename=/home/llagoeiro/Desktop/IC/IC-Prometheus-Webots/webots_prom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; collision mesh filename=/home/llagoeiro/Desktop/IC/IC-Prometheus-Webots/webots_prom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
- link peito: geometry collision mesh filename=/home/llagoeiro/Desktop/IC/IC-Prometheus-Webots/webots_prom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; collision mesh filename=/home/llagoeiro/Desktop/IC/IC-Prometheus-Webots/webots_prom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
- link pescoco: mass 0.39481195883928060786 -> 0.39481195883928055235; geometry collision mesh filename=/home/llagoeiro/Desktop/IC/IC-Prometheus-Webots/webots_prom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; collision mesh filename=/home/llagoeiro/Desktop/IC/IC-Prometheus-Webots/webots_prom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
