Commit message: Start to working with de walking

File: ros2/sigmaban_ws/src/my_package/protos/robot.urdf (robot description, URDF)
Before this commit: robot onshape, 21 links, 20 joints
Links:
- removed link braco
- removed link braco_2
- removed link canela
- removed link canela_2
- removed link capacete
- removed link conector_calcanhar
- removed link conector_calcanhar_2
- removed link joelho
- removed link joelho_2
- removed link mao
- removed link mao_2
- removed link motores_duplos
- removed link motores_duplos_2
- removed link motores_duplos_3
- removed link motores_duplos_4
- removed link ombro
- removed link ombro_2
- removed link pe_direito
- removed link pe_esquerdo
- removed link peito
- removed link pescoco
- added link body_1, mass 2.23874; collision mesh filename=body.stl; visual mesh filename=body.stl
- added link wheel_1, mass 0.335419; collision mesh filename=wheel.stl; visual mesh filename=wheel.stl
- added link wheel_2, mass 0.335419; collision mesh filename=wheel.stl; visual mesh filename=wheel.stl
Joints:
- removed joint cotovelo_direito_5
- removed joint cotovelo_esquerdo_6
- removed joint coxa_direita_11
- removed joint coxa_esquerda_12
- removed joint joelho_direito_13
- removed joint joelho_esquerdo_14
- removed joint junta_peito_pernaD_7
- removed joint junta_peito_pernaE_8
- removed joint ombro_direito_1
- removed joint ombro_direito_3
- removed joint ombro_esquerdo_2
- removed joint ombro_esquerdo_4
- removed joint pe_direito_15
- removed joint pe_direito_17
- removed joint pe_esquerdo_16
- removed joint pe_esquerdo_18
- removed joint perna_direita_9
- removed joint perna_esquerda_10
- removed joint pescoço_19
- removed joint pescoço_20
- added joint wheel1_speed: type revolute, parent body_1, child wheel_1, origin xyz=-0.02 0.0325 0.025 rpy=0 -0 0, axis -1 0 0, limit effort=1 velocity=20
- added joint wheel2_speed: type revolute, parent body_1, child wheel_2, origin xyz=0.095 0.0325 0.025 rpy=0 -0 0, axis -1 -0 -0, limit effort=1 velocity=20

File: webots/webots_prometheus/protos/robot.urdf (robot description, URDF)
Before this commit: robot onshape, 21 links, 20 joints
Links:
- link braco: geometry collision mesh filename=/home/lucas/Desktop/RoboFEI/IC/webots/webots_prometheus/bra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; collision mesh filename=/home/lucas/Desktop/RoboFEI/IC/webots/webots_prometheus/bra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
- link braco_2: geometry collision mesh filename=/home/lucas/Desktop/RoboFEI/IC/webots/webots_prometheus/bra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; collision mesh filename=/home/lucas/Desktop/RoboFEI/IC/webots/webots_prometheus/bra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
- link canela: geometry collision mesh filename=/home/lucas/Desktop/RoboFEI/IC/webots/webots_prometheus/can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; visual mesh filename=/home/lucas/Desktop/RoboFEI/IC/webots/webots_prometheus/can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
- link canela_2: geometry collision mesh filename=/home/lucas/Desktop/RoboFEI/IC/webots/webots_prometheus/can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; visual mesh filename=/home/lucas/Desktop/RoboFEI/IC/webots/webots_prometheus/can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
- link capacete: geometry collision mesh filename=/home/lucas/Desktop/RoboFEI/IC/webots/webots_prometheus/cap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; collision mesh filename=/home/lucas/Desktop/RoboFEI/IC/webots/webots_prometheus/tam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
- link conector_calcanhar: geometry collision mesh filename=/home/lucas/Desktop/RoboFEI/IC/webots/webots_prometheus/con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; visual mesh filename=/home/lucas/Desktop/RoboFEI/IC/webots/webots_prometheus/con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
- link conector_calcanhar_2: geometry collision mesh filename=/home/lucas/Desktop/RoboFEI/IC/webots/webots_prometheus/con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; visual mesh filename=/home/lucas/Desktop/RoboFEI/IC/webots/webots_prometheus/con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
- link joelho: geometry collision mesh filename=/home/lucas/Desktop/RoboFEI/IC/webots/webots_prometheus/cox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; collision mesh filename=/home/lucas/Desktop/RoboFEI/IC/webots/webots_prometheus/xm_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
- link joelho_2: geometry collision mesh filename=/home/lucas/Desktop/RoboFEI/IC/webots/webots_prometheus/cox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; collision mesh filename=/home/lucas/Desktop/RoboFEI/IC/webots/webots_prometheus/xm_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
- link mao: geometry collision mesh filename=/home/lucas/Desktop/RoboFEI/IC/webots/webots_prometheus/apo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; collision mesh filename=/home/lucas/Desktop/RoboFEI/IC/webots/webots_prometheus/apo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
- link mao_2: geometry collision mesh filename=/home/lucas/Desktop/RoboFEI/IC/webots/webots_prometheus/apo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; collision mesh filename=/home/lucas/Desktop/RoboFEI/IC/webots/webots_prometheus/apo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
- link motores_duplos: geometry collision mesh filename=/home/lucas/Desktop/RoboFEI/IC/webots/webots_prometheus/jun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; collision mesh filename=/home/lucas/Desktop/RoboFEI/IC/webots/webots_prometheus/pec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
- link motores_duplos_2: geometry collision mesh filename=/home/lucas/Desktop/RoboFEI/IC/webots/webots_prometheus/jun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; collision mesh filename=/home/lucas/Desktop/RoboFEI/IC/webots/webots_prometheus/pec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
- link motores_duplos_3: geometry collision mesh filename=/home/lucas/Desktop/RoboFEI/IC/webots/webots_prometheus/jun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; collision mesh filename=/home/lucas/Desktop/RoboFEI/IC/webots/webots_prometheus/pec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
- link motores_duplos_4: geometry collision mesh filename=/home/lucas/Desktop/RoboFEI/IC/webots/webots_prometheus/jun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; collision mesh filename=/home/lucas/Desktop/RoboFEI/IC/webots/webots_prometheus/pec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
- link ombro: geometry collision mesh filename=/home/lucas/Desktop/RoboFEI/IC/webots/webots_prometheus/omb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; visual mesh filename=/home/lucas/Desktop/RoboFEI/IC/webots/webots_prometheus/omb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
- link ombro_2: geometry collision mesh filename=/home/lucas/Desktop/RoboFEI/IC/webots/webots_prometheus/omb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; visual mesh filename=/home/lucas/Desktop/RoboFEI/IC/webots/webots_prometheus/omb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
- link pe_direito: geometry collision mesh filename=/home/lucas/Desktop/RoboFEI/IC/webots/webots_prometheus/con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; collision mesh filename=/home/lucas/Desktop/RoboFEI/IC/webots/webots_prometheus/pe.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
- link pe_esquerdo: geometry collision mesh filename=/home/lucas/Desktop/RoboFEI/IC/webots/webots_prometheus/con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; collision mesh filename=/home/lucas/Desktop/RoboFEI/IC/webots/webots_prometheus/pe.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
- link peito: geometry collision mesh filename=/home/lucas/Desktop/RoboFEI/IC/webots/webots_prometheus/bas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; collision mesh filename=/home/lucas/Desktop/RoboFEI/IC/webots/webots_prometheus/bat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
- link pescoco: geometry collision mesh filename=/home/lucas/Desktop/RoboFEI/IC/webots/webots_prometheus/pes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; collision mesh filename=/home/lucas/Desktop/RoboFEI/IC/webots/webots_prometheus/xm_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
